File: Eagle Files/CPU.sch (EAGLE design)
At the start: 29 parts, among them IC1 74HC574N, IC10 74HC574N, IC11 74LS541N, IC12 CY62256LL-PC, IC13 74AS04N, IC14 74AS04N, IC15 74S283N, IC16 74S283N, IC19 74ALS04N, IC2 74LS541N, IC20 74LS541N, IC21 74LS08N, IC3 4514N, IC4 74LS04N, IC5 74HC574N, IC6 74LS541N, IC7 CY62256LL-PC, IC8 74S283N, IC9 74S283N

Commit message: Final Schematics
Connections:
- removed net N$54: IC12G$1.A8, IC7G$1.A8
- removed net N$55: IC12G$1.A9, IC7G$1.A9
- removed net N$56: IC12G$1.A10, IC7G$1.A10
- removed net N$58: IC12G$1.A12, IC7G$1.A12
- removed net N$59: IC12G$1.A13, IC7G$1.A13
- removed net N$60: IC12G$1.A14, IC7G$1.A14
- net GND: now also IC12G$1.!CE, IC12G$1.!OE, IC12G$1.A10, IC12G$1.A12, IC12G$1.A13, IC12G$1.A14, IC12G$1.A8, IC12G$1.A9, IC7G$1.!CE, IC7G$1.!OE, IC7G$1.A10, IC7G$1.A12, IC7G$1.A13, IC7G$1.A14, IC7G$1.A8, IC7G$1.A9
- net N$46: now also IC17.Q0; no longer IC18.Q3
- net N$47: now also IC17.Q1; no longer IC18.Q2
- net N$48: now also IC17.Q2; no longer IC18.Q1
- net N$49: now also IC17.Q3; no longer IC18.Q0
- net N$50: now also IC18.Q0; no longer IC17.Q3
- net N$51: now also IC18.Q1; no longer IC17.Q2
- net N$52: now also IC18.Q2; no longer IC17.Q1
- net N$53: now also IC18.Q3; no longer IC17.Q0
- net VCC: now also IC12G$1.!WE, IC7G$1.!WE

Commit message: Final Schematics
Connections:
- new net N$54: IC12G$1.DQ0, IC20A.A1
- new net N$55: IC12G$1.DQ1, IC20A.A2
- new net N$56: IC12G$1.DQ2, IC20A.A3
- new net N$58: IC12G$1.DQ4, IC20A.A5
- new net N$59: IC12G$1.DQ5, IC20A.A6
- new net N$60: IC12G$1.DQ6, IC20A.A7
- new net N$76: IC21B.I0
- new net N$77: IC12G$1.DQ7, IC20A.A8
- net BUS0: no longer IC12G$1.DQ0, IC20A.A1
- net BUS1: no longer IC12G$1.DQ1, IC20A.A2
- net BUS2: no longer IC12G$1.DQ2, IC20A.A3
- net BUS3: no longer IC12G$1.DQ3, IC20A.A4
- net BUS4: no longer IC12G$1.DQ4, IC20A.A5
- net BUS5: no longer IC12G$1.DQ5, IC20A.A6
- net BUS6: no longer IC12G$1.DQ6, IC20A.A7
- net BUS7: no longer IC12G$1.DQ7, IC20A.A8
- net GND: now also IC12G$1.A11, IC7G$1.A11
- net N$57: now also IC12G$1.DQ3, IC20A.A4; no longer IC12G$1.A11, IC7G$1.A11
- net N$72: now also IC19A.I
