File: Eagle Files/CPU.sch (EAGLE design)
At the start: 31 parts, among them IC1 74HC574N, IC10 74HC574N, IC11 74LS541N, IC12 CY62256LL-PC, IC13 74AS04N, IC14 74AS04N, IC15 74S283N, IC16 74S283N, IC19 74ALS04N, IC2 74LS541N, IC20 74LS541N, IC21 74LS08N, IC3 4514N, IC4 74LS04N, IC5 74HC574N, IC6 74LS541N, IC7 CY62256LL-PC, IC8 74S283N, IC9 74S283N

Commit message: Added Pull-Up and Pull-Down resistors
Parts:
- removed PAD1, PAD2: WIREPAD2,54/1,0, wirepad:WIREPAD2,54/1,0
- added C1, C2: (no value), rcl:C-EU025-024X044
- added IC22: NE555, st-microelectronics:NE555
- added R1, R10, R11, R12, R13, R14, R15, R16, R17, R2, R26, R27, R28, R29, R3, R30, R31, R32, R33, R34, R35, R36, R37, R4, R5, R6, R7, R8, R9: (no value), resistor:R-US_0204/2V
- added R18, R19, R20, R21, R22, R23, R24, R25: (no value), rcl:R-US_0204/2V
Connections:
- new net N$78: IC3A.S7, R26.1
- new net N$80: IC3A.S8, R27.1
- new net N$81: IC3A.S9, R28.1
- new net N$82: IC3A.S10, R29.1
- new net N$83: IC3A.S11, R30.1
- new net N$84: IC3A.S12, R31.1
- new net N$85: IC3A.S13, R32.1
- new net N$86: IC3A.S14, R33.1
- new net N$87: IC3A.S15, R34.1
- new net N$88: C1.1, IC22.CON
- new net N$89: IC22.DIS, R35.1, R37.2
- new net N$90: C2.1, IC22.TRE, IC22.TRI, R36.1
- new net N$91: R36.2, R37.1
- net BUS0: now also R1.2
- net BUS1: now also R2.2
- net BUS2: now also R3.2
- net BUS3: now also R4.2
- net BUS4: now also R5.1
- net BUS5: now also R6.1
- net BUS6: now also R7.1
- net BUS7: now also R8.1
- net GND: now also C1.2, C2.2, IC22.GND, R1.1, R10.1, R11.1, R12.1, R13.1, R14.2, R15.2, R16.2, R17.2, R18.2, R19.2, R2.1, R20.2, R21.2, R22.1, R23.1, R24.1, R25.1, R26.2, R27.2, R28.2, R29.2, R3.1, R30.2, R31.2, R32.2, R33.2, R34.2, R4.1, R5.2, R6.2, R7.2, R8.2, R9.1; no longer PAD2.P
- net N$27: now also R17.1, R22.2
- net N$28: now also R16.1, R23.2
- net N$29: now also R15.1, R24.2
- net N$30: now also R14.1, R25.2
- net N$31: now also R13.2, R21.1
- net N$32: now also R11.2, R12.2, R20.1
- net N$33: now also IC9A.S2, R10.2, R19.1
- net N$34: now also R18.1, R9.2
- net N$70: now also IC22.OUT
- net VCC: now also IC22./RES, IC22.VCC+, R35.2; no longer PAD1.P
