File: Eagle Files/CPU.sch (EAGLE design)
At the start: 89 parts, among them IC1 74AS574N, IC10 74AC283N, IC11 74AS574N, IC12 74LS541N, IC13 74HC393N, IC14 74LS541N, IC15 74LS32N, IC16 NE555, IC18 74LS541N, IC2 74AS574N, IC3 74LS541N, IC4 74LS541N, IC5 CY62256LL-PC, IC6 CY62256LL-PC, IC7 4514N, IC8 74HC04N, IC9 74AC283N

Commit message: Ready for routing
Parts:
- added IC17: 74LS32N, 74xx-us:74LS32N
- added IC19: 74HC04N, 74xx-eu:74HC04N
- added R31, R32, R33, R34, R35, R36, R37, R38, R39, R40, R41, R42, R43, R44, R45, R46, R47: (no value), rcl:R-US_MELF0102AX
Connections:
- new net N$149: IC7A.S7, R39.2
- new net N$150: IC7A.S8, R40.2
- new net N$151: IC7A.S9, R41.2
- new net N$152: IC7A.S10, R42.2
- new net N$153: IC7A.S11, R43.2
- new net N$154: IC7A.S12, R44.2
- new net N$155: IC7A.S13, R45.2
- new net N$156: IC7A.S14, R46.2
- new net N$157: IC7A.S15, R47.2
- new net N$158: IC15C.O, IC17A.I1
- new net N$159: IC15D.O, IC17A.I0
- new net N$160: IC17A.O, IC19A.I
- new net N$162: IC13B.A, IC19A.O
- net GND: now also R31.1, R32.2, R33.2, R34.2, R35.1, R36.1, R37.1, R38.1, R39.1, R40.1, R41.1, R42.1, R43.1, R44.1, R45.1, R46.1, R47.1
- net N$107: now also R36.2
- net N$108: now also R38.2
- net N$109: now also R35.2
- net N$110: now also R33.1
- net N$111: now also R32.1
- net N$113: now also R34.1
- net N$114: now also R37.2
- net N$128: no longer IC13B.A
- net N$129: no longer IC15B.I0
- net N$132: now also IC15B.I0
- net N$19: now also IC15C.I0
- net N$20: now also IC15D.I1
- net N$21: now also IC15D.I0
- net N$62: now also IC15C.I1
- net N$96: now also R31.2
Other:
- moved on the sheet: IC13A, IC13B

Commit message: Ready for routing
Parts:
- removed IC19: 74HC04N, 74xx-eu:74HC04N
- added GND, VCC: (no value), pinhead:PINHD-1X1
Connections:
- removed net N$162: IC13B.A, IC19A.O
- net N$160: now also IC13B.A; no longer IC19A.I
Changed lines of the file:
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@@
 <part name="SUPPLY20" library="supply2" library_urn="urn:adsk.eagle:library:372" deviceset="GND" device=""/>
 <part name="IC17" library="74xx-us" library_urn="urn:adsk.eagle:library:88" deviceset="74*32" device="N" technology="LS"/>
-<part name="IC19" library="74xx-eu" library_urn="urn:adsk.eagle:library:85" deviceset="74*04" device="N" technology="HC"/>
+<part name="VCC" library="pinhead" library_urn="urn:adsk.eagle:library:325" deviceset="PINHD-1X1" device=""/>
+<part name="GND" library="pinhead" library_urn="urn:adsk.eagle:library:325" deviceset="PINHD-1X1" device=""/>
 </parts>
 <sheets>
@@
 <instance part="IC15" gate="D" x="-172.72" y="-45.72" rot="R270"/>
 <instance part="IC17" gate="A" x="-205.74" y="-66.04" rot="R180"/>
-<instance part="IC19" gate="A" x="-231.14" y="-55.88" rot="R90"/>
+<instance part="VCC" gate="G$1" x="-142.24" y="-66.04"/>
+<instance part="GND" gate="G$1" x="-142.24" y="-76.2"/>
 </instances>
 <busses>
@@
 <wire x1="-231.14" y1="-66.04" x2="-218.44" y2="-66.04" width="0.1524" layer="91"/>
 <junction x="-218.44" y="-66.04"/>
-<pinref part="IC19" gate="A" pin="I"/>
-<junction x="-231.14" y="-66.04"/>
-</segment>
-</net>
-<net name="N$162" class="0">
-<segment>
 <pinref part="IC13" gate="B" pin="A"/>
 <wire x1="-220.98" y1="-7.62" x2="-231.14" y2="-7.62" width="0.1524" layer="91"/>
 <junction x="-220.98" y="-7.62"/>
-<wire x1="-231.14" y1="-45.72" x2="-231.14" y2="-7.62" width="0.1524" layer="91"/>
-<pinref part="IC19" gate="A" pin="O"/>
-<junction x="-231.14" y="-45.72"/>
-</segment>
-</net>
+<wire x1="-231.14" y1="-66.04" x2="-231.14" y2="-7.62" width="0.1524" layer="91"/>
+</segment>
+</net>
