File: Eagle Files/CPU.brd (EAGLE design)
At the start: 210.8 x 125.4 mm, 29 parts, among them IC1 74HC574N, IC10 74HC574N, IC11 74LS541N, IC12 CY62256LL-PC, IC13 74AS04N, IC14 74AS04N, IC15 74S283N, IC16 74S283N, IC19 74ALS04N, IC2 74LS541N, IC20 74LS541N, IC21 74LS08N, IC3 4514N, IC4 74LS04N, IC5 74HC574N, IC6 74LS541N, IC7 CY62256LL-PC, IC8 74S283N, IC9 74S283N

Commit message: Final Schematics
Parts:
- moved IC6 105.4 mm to (198.1, 52.1)
- moved IC5 103.7 mm to (198.1, 26.7)
- moved IC15 57.4 mm to (215.9, 106.7)
- moved IC19 54.8 mm to (118.1, 62.2)
- moved IC9 39.9 mm to (149.9, 88.9)
- moved IC1 38.2 mm to (154.9, 50.8)
- moved IC14 29.0 mm to (214.6, 80.0)
- moved IC13 26.8 mm to (186.7, 80.0)
- moved IC21 24.7 mm to (118.1, 43.2)
- moved IC4 24.4 mm to (88.9, 72.4)
- moved IC16 24.3 mm to (186.7, 106.7)
- moved IC11 22.5 mm to (94.0, 125.7)
- moved IC10 20.3 mm to (94.0, 105.4)
- moved LED2 16.1 mm to (55.9, 104.1)
- moved LED3 16.1 mm to (49.5, 104.1)
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Connections:
- new net N$54: IC12.11, IC20.2
- new net N$55: IC12.12, IC20.3
- new net N$56: IC12.13, IC20.4
- new net N$58: IC12.16, IC20.6
- new net N$59: IC12.17, IC20.7
- new net N$60: IC12.18, IC20.8
- new net N$76: IC21.4
- new net N$77: IC12.19, IC20.9
- net BUS0: no longer IC12.11, IC20.2
- net BUS1: no longer IC12.12, IC20.3
- net BUS2: no longer IC12.13, IC20.4
- net BUS3: no longer IC12.15, IC20.5
- net BUS4: no longer IC12.16, IC20.6
- net BUS5: no longer IC12.17, IC20.7
- net BUS6: no longer IC12.18, IC20.8
- net BUS7: no longer IC12.19, IC20.9
- net GND: now also IC12.7, IC7.7
- net N$57: now also IC12.15, IC20.5; no longer IC12.7, IC7.7
- net N$72: now also IC19.1
Routing:
- net N$2: track 94.9 -> 226.3 mm, vias 2 -> 1
- net N$1: track 117.3 -> 232.0 mm
- net N$5: track 236.9 -> 131.6 mm
- net N$4: track 216.3 -> 136.1 mm, vias 2 -> 1
- net BUS4: track 540.2 -> 460.8 mm, vias 5 -> 4
- net BUS0: track 288.5 -> 367.1 mm, vias 1 -> 6
- net N$23: track 42.0 -> 117.8 mm
- net BUS5: track 557.4 -> 486.7 mm, vias 3 -> 4
- net N$30: track 101.9 -> 171.9 mm, vias 3 -> 1
- net N$25: track 123.5 -> 190.2 mm, vias 0 -> 1
- net N$67: track 177.1 -> 111.4 mm, vias 2 -> 0
- net BUS2: track 368.2 -> 427.6 mm, vias 0 -> 3
- net VCC: track 632.0 -> 690.0 mm
- net BUS7: track 547.7 -> 491.7 mm, vias 4 -> 2
- net N$77: track 0.00 -> 55.9 mm, vias 0 -> 1
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Other:
- board size 210.8 x 125.4 mm -> 274.3 x 191.4 mm

Commit message: Removed bugs
Parts:
- moved IC13 108.5 mm to (283.2, 129.5)
- moved IC16 107.4 mm to (281.9, 156.2)
- moved IC20 91.7 mm to (40.6, 118.1)
- moved IC9 78.6 mm to (217.2, 129.5)
- moved IC8 75.4 mm to (184.2, 129.5)
- moved LED8 70.1 mm to (21.6, 174.0)
- moved LED7 70.0 mm to (26.7, 174.0)
- moved LED6 69.9 mm to (31.8, 174.0)
- moved LED1 69.9 mm to (63.5, 174.0)
- moved LED2 69.9 mm to (57.1, 174.0)
- moved LED3 69.9 mm to (50.8, 174.0)
- moved LED4 69.9 mm to (44.5, 174.0)
- moved LED5 69.9 mm to (38.1, 174.0)
- moved IC14 61.7 mm to (251.5, 129.5)
- moved IC15 59.9 mm to (251.5, 154.9)
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Routing:
- net GND: track 899.7 -> 1177.4 mm
- net BUS7: track 491.7 -> 718.2 mm, vias 2 -> 1
- net VCC: track 690.0 -> 893.9 mm, vias 1 -> 4
- net BUS0: track 367.1 -> 571.0 mm
- net BUS6: track 520.5 -> 720.2 mm
- net BUS4: track 460.8 -> 632.8 mm, vias 4 -> 2
- net BUS5: track 486.7 -> 631.2 mm, vias 4 -> 3
- net N$32: track 112.3 -> 246.5 mm, vias 0 -> 3
- net BUS2: track 427.6 -> 558.0 mm, vias 3 -> 5
- net BUS1: track 459.0 -> 577.6 mm, vias 2 -> 4
- net N$31: track 112.9 -> 225.7 mm, vias 0 -> 3
- net N$62: track 112.8 -> 219.1 mm
- net N$23: track 117.8 -> 221.9 mm, vias 0 -> 1
- net BUS3: track 422.5 -> 526.2 mm, vias 3 -> 7
- net N$20: track 111.6 -> 204.4 mm, vias 1 -> 0
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Other:
- board size 274.3 x 191.4 mm -> 509.2 x 228.3 mm
